File: Project/qazimodo plate.kicad_pcb (KiCad board)
At the start: 2 copper layers, 284.8 x 94.2 mm, 0 parts

Commit message: revision work
Routing:
- net (no net): vias 0 -> 1
Other:
- board size 284.8 x 94.2 mm -> 285.8 x 95.2 mm
