File: Project/matrix.kicad_sch (KiCad schematic)
At the start: 166 parts

Commit message: matrix issues deteced and fixed, needs new silkscreen
Connections:
- net COL0: no longer MX43b1.1 (COL)
- net COL1: now also MX43b1.1 (COL); no longer MX44.1 (COL)
- net COL10: now also MX39.1 (COL), MX39b1.1 (COL), MX51a1.1 (COL), MX51b1.1 (COL); no longer MX40.1 (COL)
- net COL11: now also MX40.1 (COL); no longer MX41.1 (COL)
- net COL12: now also MX41.1 (COL); no longer MX42.1 (COL)
- net COL13: now also MX42.1 (COL); no longer MX15.1 (COL)
- net COL2: now also MX44.1 (COL); no longer MX45.1 (COL)
- net COL3: now also MX45.1 (COL); no longer MX46.1 (COL)
- net COL4: now also MX46.1 (COL); no longer MX47.1 (COL)
- net COL5: now also MX47.1 (COL); no longer MX48.1 (COL)
- net COL6: now also MX48.1 (COL); no longer MX49.1 (COL)
- net COL7: now also MX49.1 (COL); no longer MX50.1 (COL)
- net COL8: now also MX50.1 (COL); no longer MX51.1 (COL), MX51a1.1 (COL), MX51b1.1 (COL)
- net COL9: now also MX51.1 (COL); no longer MX39.1 (COL), MX39b1.1 (COL)
- net ROW0: now also D70.1 (K)
- net ROW2: no longer D70.1 (K)
- net at D51.2 (A), MX39a1.2 (ROW): no longer MX39.2 (ROW)
- net at D48.2 (A), MX39b1.2 (ROW): now also MX39.2 (ROW)
- net at D46.2 (A), MX51b1.2 (ROW): now also MX51a1.2 (ROW); no longer MX51.2 (ROW)
- net at D42.2 (A): now also MX51.2 (ROW); no longer MX51a1.2 (ROW)
- new net COL14: MX15.1 (COL)
Other:
- note removed: "MX15 here!!!"
- moved on the sheet: D1, D10, D15, D20, D25, D30, D35, D40, D42, D46, D48, D56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

Commit message: revision work
Parts:
- removed MX55a1, MX56a1, MX64a1, MX65a1: MX-NoLED, MX_Only:MXOnly-1.25U-NoLED, symbol MX_Alps_Hybrid:MX-NoLED
- removed MX55b1, MX57b1, MX63a1, MX65: MX-NoLED, MX_Only:MXOnly-1.5U-NoLED, symbol MX_Alps_Hybrid:MX-NoLED
- removed MX64c1: MX-NoLED, MX_Only:MXOnly-1U-NoLED, symbol MX_Alps_Hybrid:MX-NoLED
- MX63b1: footprint MX_Only:MXOnly-1U-NoLED -> MX_Only:MXOnly-1.25U-NoLED
Other:
- moved on the sheet: MX64, MX64b1, MX65b1

Commit message: revision work
Parts:
- D1, D10, D11, D12, D13, D14, D15, D16, D17, D18, D19, D2, D20, D21, D22, D23, D24, D25, D26, D27, D28, D29, D3, D30, D31, D32, D33, D34, D35, D36, D37, D38, D39, D4, D40, D41, D42, D43, D44, D45, D46, D47, D48, D49, D5, D50, D51, D52, D53, D54, D55, D56, D57, D58, D59, D6, D60, D61, D62, D63, D64, D65, D66, D67, D68, D69, D7, D70, D71, D8, D9: footprint Diode_SMD:D_SOD-123F -> random-keyboard-parts:D_SOD-123F(handsoldering)
